File: smk_test_board/smk_test_board.kicad_pcb (KiCad board)
At the start: 2 copper layers, 76 x 113.2 mm, 35 parts, among them J1 Battery JST-SH, SW00 KS-2P02B01-02, SW01 KS-2P02B01-02, SW10 KS-2P02B01-02, SW11 KS-2P02B01-02, SW12 KS-2P02B01-02, SW20 KS-2P02B01-02, SW21 KS-2P02B01-02, SW22 KS-2P02B01-02, U1 XIAO_ESP32C6, U2 SN74AHCT1G125DBVR

Commit message: Fix round 1: move LEDs off the switch boss, wire missing decoupling
Controller review round 1 on Task 6, both concerns confirmed real:

- LED moved from key centre to (kx, ky+5.9) -- 5.9mm south, the offset
  generate_kbd_rp2040.py:163 documents as the standard south-facing SMD
  LED position for MX-compatible/low-profile switches. Centre landed
  square on the switch's own Ø5.2mm boss NPTH, which is exactly what the
  round-1 kicad-cli DRC caught. test_leds_sit_under_their_keys replaced
  with test_leds_sit_at_the_south_facing_led_window (controller-supplied).

  Re-running DRC confirms the boss violations are gone, but a DIFFERENT
  hole_clearance violation appears in their place: at 5.9mm south, the
  LED's own pads (±2.725mm local X, unchanged from the sibling's current
  fp_sk6812mini -- confirmed byte-identical) land inside the switch's two
  Ø3.0mm LEG NPTH holes, by up to 1.31mm of real penetration, not a
  marginal clearance miss. Computed with a script before touching any
  code, then confirmed against the real kicad-cli DRC output (24 of 25
  remaining hole_clearance violations are RGBn-vs-SWrc-leg-NPTH, actual
  0.0000mm). generate_kbd_rp2040.py:163-170's "5.9mm south... confirmed
  clear of the switch's own SMD pads" is a changelog entry for an
  EARLIER, since-superseded revision of that file -- it only claims
  clearance from the SMD PADS, not the leg holes, and a later comment in
  the same file records the shipped board moved to 6.025mm NORTH instead,
  specifically because straight-south left no gap against the leg holes.
  Implemented the literal instruction (kx, ky+5.9) as given rather than
  substituting my own reading of the sibling's history; reporting the
  finding rather than silently widening anything to make it pass, per the
  round-1 instruction's own "if any remain, report".

- build_nets() now wires C1-C9 (100nF per LED, VSYS-GND) and C10/C11
  (100nF encoder debounce, ENC_A/ENC_B-GND) -- previously missing
  entirely despite being in t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
Parts:
- added C10: 100n, kbd:RC_0603, F.Cu at (57.3, 20.3)
- added C11: 100n, kbd:RC_0603, F.Cu at (68.9, 20.3)
- added C2: 100n, kbd:RC_0603, B.Cu at (48.9, 27.3)
- added C3: 100n, kbd:RC_0603, B.Cu at (67.9, 27.3)
- added C4: 100n, kbd:RC_0603, B.Cu at (29.8, 46.4)
- added C5: 100n, kbd:RC_0603, B.Cu at (48.9, 46.4)
- added C6: 100n, kbd:RC_0603, B.Cu at (67.9, 46.4)
- added C7: 100n, kbd:RC_0603, B.Cu at (29.8, 65.4)
- added C8: 100n, kbd:RC_0603, B.Cu at (48.9, 65.4)
- added C9: 100n, kbd:RC_0603, B.Cu at (67.9, 65.4)
- added C_BULK: 100u, kbd:RC_0603, F.Cu at (63.1, 104.9)
- C1: value 100u -> 100n; moved to B.Cu
- moved C1 84.4 mm to (29.8, 27.3)
- moved RGB4 5.90 mm to (25.0, 50.0)
- moved RGB5 5.90 mm to (44.0, 50.0)
- moved RGB6 5.90 mm to (63.1, 50.0)
- moved RGB1 5.90 mm to (25.0, 30.9)
- moved RGB2 5.90 mm to (44.0, 30.9)
- moved RGB3 5.90 mm to (63.1, 30.9)
- moved RGB7 5.90 mm to (25.0, 69.0)
- moved RGB8 5.90 mm to (44.0, 69.0)
- moved RGB9 5.90 mm to (63.1, 69.0)

Commit message: Fix round 2: LEDs to the real north window, obstacle-driven cap search
Controller review round 2 on Task 6, both concerns confirmed real and
fixed at the root rather than by hand.

- LED offset corrected from 5.9mm south to -6.025mm north
  (kx, ky-6.025). Round 1 quoted generate_kbd_rp2040.py:163-170's prose
  changelog entry ("5.9mm south... confirmed clear of the switch's own
  SMD pads"), which turned out to describe an earlier, since-superseded
  attempt -- the code that file actually ships (:2050-2059,
  LED_OFFSET_Y = -6.025) moved north after finding south left the LED's
  own pads on the same side as the switch's leg NPTH holes, "no matter
  how it was routed". test_leds_sit_at_the_south_facing_led_window
  replaced with test_leds_sit_at_the_north_led_window
  (controller-supplied).

- The C3-vs-ENC1 clearance shortfall is fixed by making the cap-position
  search itself obstacle-aware instead of nudging C3's number: added
  _pad_obstacles()/_probe_obstacles() (read a footprint's own emitted
  pad/hole geometry back out, the same technique
  _socket_back_courtyard() already used for the Gateron's courtyard, now
  generalized to any footprint built from gm's pad()/npth()) and
  _best_clear_offset()/_cap_offsets_near() (grid-search the nearest safe
  position near a target point). build_pcb() now picks the Gateron's
  obstacle set or the EC11's, whichever is actually at that key, before
  placing each per-LED cap -- so row0/col2's cap is checked against the
  EC11 it actually sits next to, not a socket that isn't there.

  Two real bugs surfaced and fixed while building this:
  (1) the search's first version maximized clearance over the whole
  search box rather than finding the nearest point that merely clears a
  safety margin, so it had no reason to stay near the LED at all and
  reliably ran to the box's far edge -- caught by
  test_no_unexpected_courtyard_overlaps when a cap fled 6mm north into
  the PREVIOUS row's own switch courtyard, a neighbour its o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
Parts:
- moved C11 13.8 mm to (63.1, 32.8)
- moved C7 12.5 mm to (25.0, 53.9)
- moved C8 12.5 mm to (44.0, 53.9)
- moved C9 12.5 mm to (63.1, 53.9)
- moved C2 12.5 mm to (44.0, 15.8)
- moved C3 12.5 mm to (63.1, 15.8)
- moved C1 12.5 mm to (25.0, 15.8)
- moved C5 12.5 mm to (44.0, 34.8)
- moved C6 12.5 mm to (63.1, 34.8)
- moved C4 12.5 mm to (25.0, 34.8)
- moved RGB4 11.9 mm to (25.0, 38.0)
- moved RGB5 11.9 mm to (44.0, 38.0)
- moved RGB6 11.9 mm to (63.1, 38.0)
- moved RGB1 11.9 mm to (25.0, 19.0)
- moved RGB2 11.9 mm to (44.0, 19.0)
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Changed lines of the file:
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@@
   )
   (footprint "smk_test_board:SK6812MINI_E" (layer "B.Cu")
-  (at 25 30.9 180)
+  (at 25 18.975 180)
   (property "Reference" "RGB1" (at 0 2.6 180) (layer "B.SilkS")
     (effects (font (size 1 1) (thickness 0.15)) (justify mirror))
@@
   )
   (footprint "kbd:RC_0603" (layer "B.Cu")
-  (at 29.8 27.3)
+  (at 25 15.775)
   (property "Reference" "C1" (at 0 -1.5 0) (layer "B.SilkS")
     (effects (font (size 1 1) (thickness 0.15)) (justify mirror))
@@
   )
   (footprint "smk_test_board:SK6812MINI_E" (layer "B.Cu")
-  (at 44.05 30.9 180)
+  (at 44.05 18.975 180)
   (property "Reference" "RGB2" (at 0 2.6 180) (layer "B.SilkS")
     (effects (font (size 1 1) (thickness 0.15)) (justify mirror))
@@
   )
   (footprint "kbd:RC_0603" (layer "B.Cu")
-  (at 48.85 27.3)
+  (at 44.05 15.775)
   (property "Reference" "C2" (at 0 -1.5 0) (layer "B.SilkS")
     (effects (font (size 1 1) (thickness 0.15)) (justify mirror))
@@
   )
   (footprint "kbd:RC_0603" (layer "F.Cu")
-  (at 57.3 20.3)
+  (at 63.1 17.2)
   (property "Reference" "C10" (at 0 -1.5 0) (layer "F.SilkS")
     (effects (font (size 1 1) (thickness 0.15)))
@@
   )
   (footprint "kbd:RC_0603" (layer "F.Cu")
-  (at 68.9 20.3)
+  (at 63.1 32.8)
   (property "Reference" "C11" (at 0 -1.5 0) (layer "F.SilkS")
     (effects (font (size 1 1) (thickness 0.15)))
@@
   )
   (footprint "smk_test_board:SK6812MINI_E" (layer "B.Cu")
-  (at 63.1 30.9 180)
+  (at 63.1 18.975 180)
   (property "Reference" "RGB3" (at 0 2.6 180) (layer "B.SilkS")
     (effects (font (size 1 1) (thickness 0.15)) (justify mirror))
@@
   )
   (footprint "kbd:RC_0603" (layer "B.Cu")
-  (at 67.9 27.3)
+  (at 63.1 15.775)
   (property "Reference" "C3" (at 0 -1.5 0) (layer "B.SilkS")
     (effects (font (size 1 1) (thickness 0.15)) (justify mirror))
@@
   )
   (footprint "smk_test_board:SK6812MINI_E" (layer "B.Cu")
-  (at 25 49.95 180)
+  (at 25 38.025 180)
   (property "Reference" "RGB4" (at 0 2.6 180) (layer "B.SilkS")
     (effects (font (size 1 1) (thickness 0.15)) (justify mirror))
@@
   )
   (footprint "kbd:RC_0603" (layer "B.Cu")
-  (at 29.8 46.35)
+  (at 25 34.825)
   (property "Reference" "C4" (at 0 -1.5 0) (layer "B.SilkS")
     (effects (font (size 1 1) (thickness 0.15)) (justify mirror))
@@
   )
   (footprint "smk_test_board:SK6812MINI_E" (layer "B.Cu")
-  (at 44.05 49.95 180)
+  (at 44.05 38.025 180)
   (property "Reference" "RGB5" (at 0 2.6 180) (layer "B.SilkS")
     (effects (font (size 1 1) (thickness 0.15)) (justify mirror))
@@
   )
   (footprint "kbd:RC_0603" (layer "B.Cu")
-  (at 48.85 46.35)
+  (at 44.05 34.825)
   (property "Reference" "C5" (at 0 -1.5 0) (layer "B.SilkS")
     (effects (font (size 1 1) (thickness 0.15)) (justify mirror))
@@
   )
   (footprint "smk_test_board:SK6812MINI_E" (layer "B.Cu")
-  (at 63.1 49.95 180)
+  (at 63.1 38.025 180)
   (property "Reference" "RGB6" (at 0 2.6 180) (layer "B.SilkS")
     (effects (font (size 1 1) (thickness 0.15)) (justify mirror))
@@
   )
   (footprint "kbd:RC_0603" (layer "B.Cu")
-  (at 67.9 46.35)
+  (at 63.1 34.825)
   (property "Reference" "C6" (at 0 -1.5 0) (layer "B.SilkS")
     (effects (font (size 1 1) (thickness 0.15)) (justify mirror))
@@
   )
   (footprint "smk_test_board:SK6812MINI_E" (layer "B.Cu")
-  (at 25 69 180)
+  (at 25 57.075 180)
   (property "Reference" "RGB7" (at 0 2.6 180) (layer "B.SilkS")
     (effects (font (size 1 1) (thickness 0.15)) (justify mirror))
@@
   )
   (footprint "kbd:RC_0603" (layer "B.Cu")
-  (at 29.8 65.4)
+  (at 25 53.875)
   (property "Reference" "C7" (at 0 -1.5 0) (layer "B.SilkS")
     (effects (font (size 1 1) (thickness 0.15)) (justify mirror))
@@
   )
   (footprint "smk_test_board:SK6812MINI_E" (layer "B.Cu")
-  (at 44.05 69 180)
+  (at 44.05 57.075 180)
   (property "Reference" "RGB8" (at 0 2.6 180) (layer "B.SilkS")
     (effects (font (size 1 1) (thickness 0.15)) (justify mirror))
@@
   )
   (footprint "kbd:RC_0603" (layer "B.Cu")
-  (at 48.85 65.4)
+  (at 44.05 53.875)
   (property "Reference" "C8" (at 0 -1.5 0) (layer "B.SilkS")
     (effects (font (size 1 1) (thickness 0.15)) (justify mirror))
@@
   )
   (footprint "smk_test_board:SK6812MINI_E" (layer "B.Cu")
-  (at 63.1 69 180)
+  (at 63.1 57.075 180)
   (property "Reference" "RGB9" (at 0 2.6 180) (layer "B.SilkS")
     (effects (font (size 1 1) (thickness 0.15)) (justify mirror))
@@
   )
   (footprint "kbd:RC_0603" (layer "B.Cu")
-  (at 67.9 65.4)
+  (at 63.1 53.875)
   (property "Reference" "C9" (at 0 -1.5 0) (layer "B.SilkS")
     (effects (font (size 1 1) (thickness 0.15)) (justify mirror))
