File: smk_test_board/smk_test_board.kicad_pcb (KiCad board)
At the start: 2 copper layers, 76 x 113.2 mm, 46 parts, among them J1 Battery JST-SH, SW00 KS-2P02B01-02, SW01 KS-2P02B01-02, SW10 KS-2P02B01-02, SW11 KS-2P02B01-02, SW12 KS-2P02B01-02, SW20 KS-2P02B01-02, SW21 KS-2P02B01-02, SW22 KS-2P02B01-02, U1 XIAO_ESP32C6, U2 SN74AHCT1G125DBVR

Commit message: Fix round 2: serpentine LED chain order, tg: dead-end in bring-up
Finding 1 (hardware defect): the LED chain was wired raster
(i = r*COLS+c+1), but firmware's ledChainIndex() (SMKCore/
LEDChainMapping.swift), which RGBLighting.swift actually indexes at
runtime, is serpentine -- even rows col0->COLS-1, odd rows reversed.
On this 3x3 board only row 1 disagrees between the two formulas (rows
0/2 coincide), which is why it passed review for several rounds.
Fixed generate_test_board.py's chain-index formula to match
ledChainIndex exactly, regenerated the schematic/PCB (only RGB4/C4 and
RGB6/C6 trade places; nothing else moves), and added a dedicated test
that checks all 9 positions against the transcribed formula so a
same-on-two-rows regression like this can't hide again. Also
decoupled test_leds_sit_at_the_north_led_window from the chain-index
formula (it now looks refs up via POS_OF_REF instead of computing a
ref name), so it isn't itself a second copy of the bug to keep in
sync. DRC re-run: 16 errors / 86 unconnected (errors-only), 135 / 86
(full) -- identical to docs/fabrication.md's table, same per-category
breakdown; no table update needed. Re-exported gerbers/zip locally
(gitignored, not committed) to confirm export_fab.py still runs clean
against the regenerated board.

Finding 2 (doc defect): bring-up.md's Step 5a remapped only layer 0's
tg:1 cell, leaving layer 1's mirror cell as an ordinary keycode
(key:f8) instead of trans. LayerEngine.getAction only falls through to
a lower layer on a literal trans, so the second press of the tg: key
would type F8 instead of toggling back -- no keyboard-only way off
layer 1. Step 5a now remaps both cells (mirroring the mo:1/trans
pairing already correct at row0/col2), and step 5d spells out what a
missed layer-1 edit looks like.

Minor: step 1c now names its probe points (XIAO's U1 pin 12/13) the
way 1b already did, and notes that pin is deliberately left unwired
in build_nets() (nothing on this board consumes regulated 3.3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
Parts:
- moved C4 38.1 mm to (63.1, 34.8)
- moved C6 38.1 mm to (25.0, 34.8)
- moved RGB4 38.1 mm to (63.1, 38.0)
- moved RGB6 38.1 mm to (25.0, 38.0)
Changed lines of the file:
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@@
   (footprint "smk_test_board:SK6812MINI_E" (layer "B.Cu")
   (at 25 38.025 180)
-  (property "Reference" "RGB4" (at 0 2.6 180) (layer "B.SilkS")
+  (property "Reference" "RGB6" (at 0 2.6 180) (layer "B.SilkS")
     (effects (font (size 1 1) (thickness 0.15)) (justify mirror))
   )
@@
   (attr smd)
     (pad "1" smd roundrect (at -2.725 -0.75) (size 1.35 0.82) (layers "B.Cu" "B.Mask" "B.Paste") (net 18 "VSYS") (roundrect_rratio 0.25))
-    (pad "2" smd roundrect (at -2.725 0.75) (size 1.35 0.82) (layers "B.Cu" "B.Mask" "B.Paste") (net 22 "LEDD5") (roundrect_rratio 0.25))
+    (pad "2" smd roundrect (at -2.725 0.75) (size 1.35 0.82) (layers "B.Cu" "B.Mask" "B.Paste") (net 24 "LEDD7") (roundrect_rratio 0.25))
     (pad "3" smd roundrect (at 2.725 0.75) (size 1.35 0.82) (layers "B.Cu" "B.Mask" "B.Paste") (net 16 "GND") (roundrect_rratio 0.25))
-    (pad "4" smd roundrect (at 2.725 -0.75) (size 1.35 0.82) (layers "B.Cu" "B.Mask" "B.Paste") (net 21 "LEDD4") (roundrect_rratio 0.25))
+    (pad "4" smd roundrect (at 2.725 -0.75) (size 1.35 0.82) (layers "B.Cu" "B.Mask" "B.Paste") (net 23 "LEDD6") (roundrect_rratio 0.25))
     (fp_line (start 3.65 1.875) (end 3.65 -1.875) (stroke (width 0.15) (type solid)) (layer "B.SilkS"))
     (fp_line (start 3.65 -1.875) (end -2.925 -1.875) (stroke (width 0.15) (type solid)) (layer "B.SilkS"))
@@
   (footprint "kbd:RC_0603" (layer "B.Cu")
   (at 25 34.825)
-  (property "Reference" "C4" (at 0 -1.5 0) (layer "B.SilkS")
+  (property "Reference" "C6" (at 0 -1.5 0) (layer "B.SilkS")
     (effects (font (size 1 1) (thickness 0.15)) (justify mirror))
   )
@@
   (footprint "smk_test_board:SK6812MINI_E" (layer "B.Cu")
   (at 63.1 38.025 180)
-  (property "Reference" "RGB6" (at 0 2.6 180) (layer "B.SilkS")
+  (property "Reference" "RGB4" (at 0 2.6 180) (layer "B.SilkS")
     (effects (font (size 1 1) (thickness 0.15)) (justify mirror))
   )
@@
   (attr smd)
     (pad "1" smd roundrect (at -2.725 -0.75) (size 1.35 0.82) (layers "B.Cu" "B.Mask" "B.Paste") (net 18 "VSYS") (roundrect_rratio 0.25))
-    (pad "2" smd roundrect (at -2.725 0.75) (size 1.35 0.82) (layers "B.Cu" "B.Mask" "B.Paste") (net 24 "LEDD7") (roundrect_rratio 0.25))
+    (pad "2" smd roundrect (at -2.725 0.75) (size 1.35 0.82) (layers "B.Cu" "B.Mask" "B.Paste") (net 22 "LEDD5") (roundrect_rratio 0.25))
     (pad "3" smd roundrect (at 2.725 0.75) (size 1.35 0.82) (layers "B.Cu" "B.Mask" "B.Paste") (net 16 "GND") (roundrect_rratio 0.25))
-    (pad "4" smd roundrect (at 2.725 -0.75) (size 1.35 0.82) (layers "B.Cu" "B.Mask" "B.Paste") (net 23 "LEDD6") (roundrect_rratio 0.25))
+    (pad "4" smd roundrect (at 2.725 -0.75) (size 1.35 0.82) (layers "B.Cu" "B.Mask" "B.Paste") (net 21 "LEDD4") (roundrect_rratio 0.25))
     (fp_line (start 3.65 1.875) (end 3.65 -1.875) (stroke (width 0.15) (type solid)) (layer "B.SilkS"))
     (fp_line (start 3.65 -1.875) (end -2.925 -1.875) (stroke (width 0.15) (type solid)) (layer "B.SilkS"))
@@
   (footprint "kbd:RC_0603" (layer "B.Cu")
   (at 63.1 34.825)
-  (property "Reference" "C6" (at 0 -1.5 0) (layer "B.SilkS")
-    (effects (font (size 1 1) (thickness 0.15)) (justify mirror))
-  )
+  (property "Reference" "C4" (at 0 -1.5 0) (layer "B.SilkS")
+    (effects (font (size 1 1) (thickness 0.15)) (justify mirror))
+  )
