File: smk_test_board/smk_test_board.kicad_sch (KiCad schematic)
At the start: 30 parts, among them J1 JST-PH-2 (battery), SW00 Gateron KS-33 hot-swap, SW01 Gateron KS-33 hot-swap, SW10 Gateron KS-33 hot-swap, SW11 Gateron KS-33 hot-swap, SW12 Gateron KS-33 hot-swap, SW20 Gateron KS-33 hot-swap, SW21 Gateron KS-33 hot-swap, SW22 Gateron KS-33 hot-swap, U1 Seeed XIAO ESP32-C6, U2 LEVEL SHIFTER (part TBD; VCC/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

Commit message: Fix diode polarity, drop +3V3, wire U2 as the real level shifter
Controller review round 1 on Task 5, all three self-review concerns
confirmed real:

- PAD_MAP had D_SOD-123_Back's A/K pads backwards (settled from the
  sibling's fp_diode(ref, x, y, rot, n_k, n_a, ...), which takes the
  cathode net first -- pad 1 = K, pad 2 = A). Fixed the map and flipped
  the diode's schematic instance placement to rot=180 so it still reads
  correctly on the sheet (net topology was never wrong, since labels
  attach by pin number; only the pin-to-side mapping needed to flip).
- Removed the +3V3 net outright instead of padding it to two members --
  nothing on this board actually consumes regulated 3.3V now that the
  level shifter is a VSYS-rail part. Added a general
  test_no_net_has_fewer_than_two_members() so this class of bug can't
  recur silently for any net.
- Wired U2 as the real SN74AHCT1G125DBVR (SOT-23-5), the same part the
  sibling keyboard project uses: OE#->GND (enabled), A->LEDD0, GND->GND,
  Y->LEDD1, VCC->VSYS. Copied the SOT-23-5 footprint from
  SMK_macro_pad/smk_macropad_mini/kbd.pretty and added it to
  test_footprints.py's EXPECTED.

9 tests pass. Schematic re-verified with gm.check_parens (end=0, min=0)
and kicad-cli ERC (no new multiple_net_names collisions from the diode
rotation or the level shifter's wider footprint).

Co-Authored-By: Claude Opus 5 (1M context) <noreply@anthropic.com>
Claude-Session: https://claude.ai/code/session_01RrNSSSsf75egXawfTDj93k
Parts:
- U2: value LEVEL SHIFTER (part TBD; VCC/GND/OE# not modeled) -> SN74AHCT1G125DBVR; footprint (none) -> smk_test_board:SOT-23-5
Connections:
- net GND: now also U2.1 (OE#), U2.3 (GND)
- net LEDD0: now also U2.2 (A); no longer U2.IN
- net LEDD1: now also U2.4 (Y); no longer U2.OUT
- net ROW0: now also D00.1 (K), D01.1 (K), D02.1 (K); no longer D00.2 (K), D01.2 (K), D02.2 (K)
- net ROW1: now also D10.1 (K), D11.1 (K), D12.1 (K); no longer D10.2 (K), D11.2 (K), D12.2 (K)
- net ROW2: now also D20.1 (K), D21.1 (K), D22.1 (K); no longer D20.2 (K), D21.2 (K), D22.2 (K)
- net SW02_N: now also D02.2 (A); no longer D02.1 (A)
- net VSYS: now also U2.5 (VCC)
- net at SW11.2: now also D11.2 (A); no longer D11.1 (A)
- net at SW21.2: now also D21.2 (A); no longer D21.1 (A)
- net at SW01.2: now also D01.2 (A); no longer D01.1 (A)
- net at SW00.2: now also D00.2 (A); no longer D00.1 (A)
- net at SW20.2: now also D20.2 (A); no longer D20.1 (A)
- net at SW22.2: now also D22.2 (A); no longer D22.1 (A)
- net at SW12.2: now also D12.2 (A); no longer D12.1 (A)
- net at SW10.2: now also D10.2 (A); no longer D10.1 (A)
- net +3V3: no longer names the net of U1.12 (+3V3)
- no-connect marks 4 -> 5
Other:
- moved on the sheet: D00, D01, D02, D10, D11, D12, D20, D21, D22

Commit message: Wire the battery to the XIAO, add the VBAT divider, complete the schematic
Three defects with one shape: parts that build_nets()/build_pcb() should
have carried and didn't, or carried and never told the schematic about.

1. The battery never reached the XIAO.
   J1 (the JST cell connector) fed VSYS, and VSYS fed the nine SK6812 VDD
   pins, C1-C9, C_BULK and U2's VCC -- but nothing tied VSYS to U1. The
   board could not run untethered, the XIAO's onboard charger was never in
   circuit with the cell, and on USB with no cell fitted the whole LED
   chain and the level shifter were unpowered.

   The XIAO's BAT+/BAT- are solder pads on the module's UNDERSIDE and it
   seats on female headers, so no PCB pad can mate with them:
   XIAO_ESP32C6_HEADERS is 14 pads with no BAT pad, and that is correct.
   Added J2, a labelled 2-pin THROUGH-HOLE pad pair beside U1 for two
   short flying leads the user solders to the module's underside pads.

   THT, not SMD -- these take hand-soldered wire and an SMD pad tears off.
   Polarity is made unmistakable four ways (a reversed lead puts a Li-ion
   cell backwards into the XIAO): pad 1 is the square pin-1 pad, both pads
   carry "BAT+"/"BAT-" silk, a drawn silk "+" sits outboard of pad 1 and a
   drawn "-" outboard of pad 2.

   Placement is searched, not hand-picked: _placed_obstacles() reads every
   already-placed footprint's real courtyard out of gm.FPBOX in absolute
   board coordinates, and the search demands 1.5mm of clearance -- U1's
   courtyard is larger than the module's own 21 x 17.5mm body, so clearing
   it by 1.5mm is 1.5mm of open board beyond the seated module, enough for
   an iron tip and a wire. An assert refuses to place J2 without it. Board
   outline is unchanged at 76.0 x 113.16mm.

2. VBAT sense was unwired, and the spec's premise for that was wrong.
   PIN["VBAT_SENSE"] existed and drew a schematic port, but build_nets()
   referenced it zero times -- U1 pad 1 floated while firmware read
   ADC1_CH0 as a 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
Parts:
- added C1, C10, C11, C12, C2, C3, C4, C5, C6, C7, C8, C9: 100n, smk_test_board:RC_0603, symbol kbd:C_kbd
- added C_BULK: 100u, smk_test_board:RC_0603, symbol kbd:C_kbd
- added J2: BAT+ / BAT- flying leads, smk_test_board:BAT_WIRE_PADS, symbol kbd:Conn_BAT2_tb
- added R1, R2: 200k, smk_test_board:RC_0603, symbol kbd:R_kbd
Connections:
- net ENC_A: now also C10.1
- net ENC_B: now also C11.1
- net GND: now also C1.2, C10.2, C11.2, C12.2, C2.2, C3.2, C4.2, C5.2, C6.2, C7.2, C8.2, C9.2, C_BULK.2, J2.2 (BAT-), R2.2
- net VSYS: now also C1.1, C12.1, C2.1, C3.1, C4.1, C5.1, C6.1, C7.1, C8.1, C9.1, C_BULK.1, J2.1 (BAT+), R1.1
- net VBAT_SENSE: now reaches U1.1 (VBAT_SENSE)
- net VBAT_SENSE: now also R1.2, R2.1
- no-connect marks 5 -> 4
Other:
- note added: "J2 (in PASSIVES) is the pad pair for the two flying leads soldered to the XIAO module's UNDERSIDE BAT+/BAT- pads. The XIAO sits on female headers and its battery terminals are on its bottom face, so no PCB pad can mate with them; without J2 the VSYS rail J1 feeds never reaches the module at all."
- note added: "PASSIVES (LED/encoder/shifter decoupling, bulk, VBAT sense divider)"
- note added: "POWER (JST battery input + BAT flying leads to the XIAO)"
- note removed: "POWER (JST battery input)"

Commit message: Fix battery connector BOM/schematic naming: JST-PH -> JST-SH
The board's footprint (JST_SH_SM02B_2pin_Back) has always been JST SH,
1.0mm pitch, but the BOM, spec, bring-up doc, and the schematic's own
symbol/instance value strings all said "JST-PH" (2.0mm pitch) -- a
different, incompatible connector. Someone following the BOM would order
a PH connector and a cell with a PH pigtail, and neither would fit.

Corrects every JST-PH mention to JST SH (SM02B-SRSS-TB or equivalent),
and adds a prominent BOM-area note in fabrication.md: single-cell Li-ion
pouch cells commonly ship with a JST-PH 2.0mm pigtail that will not mate
with this board's SH connector, so the buyer needs an SH-pigtail cell, a
PH-to-SH adapter, or to re-terminate.

Regenerating produces a byte-identical .kicad_pcb -- only the schematic's
two Value property strings change, confirming no electrical/geometric
change.

Co-Authored-By: Claude Opus 5 (1M context) <noreply@anthropic.com>
Claude-Session: https://claude.ai/code/session_01RrNSSSsf75egXawfTDj93k
Parts:
- J1: value JST-PH-2 (battery) -> JST-SH-2 (battery)
Changed lines of the file:
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@@
     (exclude_from_sim no) (in_bom yes) (on_board yes) (dnp no) (fields_autoplaced yes)
     (property "Reference" "J1" (at 40.64 233.68 0) (effects (font (size 1.27 1.27))))
-    (property "Value" "JST-PH-2 (battery)" (at 40.64 243.84 0) (effects (font (size 1.27 1.27))))
+    (property "Value" "JST-SH-2 (battery)" (at 40.64 243.84 0) (effects (font (size 1.27 1.27))))
     (property "Footprint" "smk_test_board:JST_SH_SM02B_2pin_Back" (at 40.64 238.76 0) (effects (font (size 1.27 1.27)) (hide yes)))
     (property "Datasheet" "~" (at 40.64 238.76 0) (effects (font (size 1.27 1.27)) (hide yes)))

Commit message: Route the board: router.py generates the copper; shrink to 65.7 x 91.73 mm
router.py rasterises every obstacle onto a 0.2 mm grid and routes with an
8-direction A* (turn and via costs), shortest MST edge first; GND is a pour
on both layers with a stub via per pad. The outline is now derived from the
placement. DRC with --refill-zones: 16 errors / 0 unconnected, as unrouted.
28 tests pass.

Co-Authored-By: Claude Opus 5.5 <noreply@anthropic.com>
Claude-Session: https://claude.ai/code/session_01PWVS4DMn5rniJecYgbPE6J
Parts:
- renumbered C_BULK to C_BULK1
